Commit message: urdf limits , velocity exp reward

File: urdf/biped_v4.urdf (robot description, URDF)
Before this commit: robot biped_v4, 47 links, 46 joints
Joints:
- joint left_hip1: limit lower=-1.732 upper=1.732 effort=3.7 velocity=10 -> lower=0 upper=0.3 effort=3.7 velocity=1
- joint right_hip1: limit lower=-1.732 upper=1.732 effort=3.7 velocity=10 -> lower=-0.3 upper=0 effort=3.7 velocity=10

Commit message: refined rewards, remover angular velocity

File: urdf/biped_v4.urdf (robot description, URDF)
Before this commit: robot biped_v4, 47 links, 46 joints
Joints:
- joint left_ankle: limit lower=-1.732 upper=1.732 effort=1.5 velocity=10 -> lower=-1.732 upper=1.732 effort=1.5 velocity=3
- joint left_hip2: limit lower=-1.732 upper=1.732 effort=3.7 velocity=10 -> lower=-1.732 upper=1.732 effort=3.7 velocity=4
- joint left_knee: limit lower=-2 upper=2 effort=5 velocity=10 -> lower=-2 upper=2 effort=5 velocity=4
- joint right_ankle: limit lower=-1.732 upper=1.732 effort=1.5 velocity=10 -> lower=-1.732 upper=1.732 effort=1.5 velocity=3
- joint right_hip1: limit lower=-0.3 upper=0 effort=3.7 velocity=10 -> lower=-0.3 upper=0 effort=3.7 velocity=1
- joint right_hip2: limit lower=-1.732 upper=1.732 effort=3.7 velocity=10 -> lower=-1.732 upper=1.732 effort=3.7 velocity=4
- joint right_knee: limit lower=-2 upper=2 effort=5 velocity=10 -> lower=-2 upper=2 effort=5 velocity=4
- joint torso: limit lower=-1.732 upper=1.732 effort=13 velocity=10 -> lower=-1.0 upper=1.0 effort=13 velocity=5

Commit message: control and domain randomisation

File: urdf/biped_v4.urdf (robot description, URDF)
Before this commit: robot biped_v4, 47 links, 46 joints
Joints:
- joint left_ankle: limit lower=-1.732 upper=1.732 effort=1.5 velocity=3 -> lower=-1.732 upper=1.732 effort=1.5 velocity=4
- joint left_hip1: limit lower=0 upper=0.3 effort=3.7 velocity=1 -> lower=0 upper=0.3 effort=3.7 velocity=4
- joint right_ankle: limit lower=-1.732 upper=1.732 effort=1.5 velocity=3 -> lower=-1.732 upper=1.732 effort=1.5 velocity=4
- joint right_hip1: limit lower=-0.3 upper=0 effort=3.7 velocity=1 -> lower=-0.3 upper=0 effort=3.7 velocity=4
- joint torso: limit lower=-1.0 upper=1.0 effort=13 velocity=5 -> lower=-1.0 upper=1.0 effort=13 velocity=4

Commit message: error correct try (being slow)

File: urdf/biped_v4.urdf (robot description, URDF)
Before this commit: robot biped_v4, 47 links, 46 joints
Joints:
- joint left_ankle: limit lower=-1.732 upper=1.732 effort=1.5 velocity=4 -> lower=-1.732 upper=1.732 effort=1 velocity=2
- joint left_hip1: limit lower=0 upper=0.3 effort=3.7 velocity=4 -> lower=0 upper=0.3 effort=1.5 velocity=2
- joint left_hip2: limit lower=-1.732 upper=1.732 effort=3.7 velocity=4 -> lower=-1.732 upper=1.732 effort=1.5 velocity=2
- joint left_knee: limit lower=-2 upper=2 effort=5 velocity=4 -> lower=-2 upper=2 effort=1.5 velocity=2
- joint right_ankle: limit lower=-1.732 upper=1.732 effort=1.5 velocity=4 -> lower=-1.732 upper=1.732 effort=1 velocity=2
- joint right_hip1: limit lower=-0.3 upper=0 effort=3.7 velocity=4 -> lower=-0.3 upper=0 effort=1.5 velocity=2
- joint right_hip2: limit lower=-1.732 upper=1.732 effort=3.7 velocity=4 -> lower=-1.732 upper=1.732 effort=1.5 velocity=2
- joint right_knee: limit lower=-2 upper=2 effort=5 velocity=4 -> lower=-2 upper=2 effort=1.5 velocity=2
- joint torso: limit lower=-1.0 upper=1.0 effort=13 velocity=4 -> lower=-1.0 upper=1.0 effort=1.8 velocity=1.8

Commit message: without torso first

File: urdf/biped_v4.urdf (robot description, URDF)
Before this commit: robot biped_v4, 47 links, 46 joints
Links:
- removed link fix_cfpipe1tobaselink
- removed link fix_cfpipe2tobaselink
- removed link fix_torsolink1
- removed link fix_torsolink2
- removed link fix_torsolink3
- removed link fix_torsotobaselink1
- removed link fix_torsotobaselink2
- removed link fix_torsoweight
- removed link servo1
- removed link world
- added link cfpipebase1, mass 0.007; collision mesh filename=/home/samaksh/biped_dev/RLstuff/Rocon-Biped-Genesis/urdf/me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; visual mesh filename=/home/samaksh/biped_dev/RLstuff/Rocon-Biped-Genesis/urdf/me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
- added link cfpipebase2, mass 0.007; collision mesh filename=/home/samaksh/biped_dev/RLstuff/Rocon-Biped-Genesis/urdf/me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; visual mesh filename=/home/samaksh/biped_dev/RLstuff/Rocon-Biped-Genesis/urdf/me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
- added link fixed_left_sensor_motor, mass 0.02; collision mesh filename=/home/samaksh/biped_dev/RLstuff/Rocon-Biped-Genesis/urdf/me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; visual mesh filename=/home/samaksh/biped_dev/RLstuff/Rocon-Biped-Genesis/urdf/me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
- added link fixed_right_sensor_motor, mass 0.02; collision mesh filename=/home/samaksh/biped_dev/RLstuff/Rocon-Biped-Genesis/urdf/me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; visual mesh filename=/home/samaksh/biped_dev/RLstuff/Rocon-Biped-Genesis/urdf/me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
- added link revolute_left_sensorstick, mass 0.003; collision mesh filename=/home/samaksh/biped_dev/RLstuff/Rocon-Biped-Genesis/urdf/me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; visual mesh filename=/home/samaksh/biped_dev/RLstuff/Rocon-Biped-Genesis/urdf/me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
- added link revolute_right_sensorstick, mass 0.003; collision mesh filename=/home/samaksh/biped_dev/RLstuff/Rocon-Biped-Genesis/urdf/me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; visual mesh filename=/home/samaksh/biped_dev/RLstuff/Rocon-Biped-Genesis/urdf/me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
- link base_link: geometry collision mesh filename=/home/samaksh/biped_dev/RLstuff/Rocon-Biped-Genesis/urdf/me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; visual mesh filename=/home/samaksh/biped_dev/RLstuff/Rocon-Biped-Genesis/urdf/me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
- link fix_femur1_3: geometry collision mesh filename=/home/samaksh/biped_dev/RLstuff/Rocon-Biped-Genesis/urdf/me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; visual mesh filename=/home/samaksh/biped_dev/RLstuff/Rocon-Biped-Genesis/urdf/me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
- link fix_femur1_4: geometry collision mesh filename=/home/samaksh/biped_dev/RLstuff/Rocon-Biped-Genesis/urdf/me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; visual mesh filename=/home/samaksh/biped_dev/RLstuff/Rocon-Biped-Genesis/urdf/me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
- link fix_left_femur2_2: geometry collision mesh filename=/home/samaksh/biped_dev/RLstuff/Rocon-Biped-Genesis/urdf/me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; visual mesh filename=/home/samaksh/biped_dev/RLstuff/Rocon-Biped-Genesis/urdf/me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
- link fix_left_femur2_3: geometry collision mesh filename=/home/samaksh/biped_dev/RLstuff/Rocon-Biped-Genesis/urdf/me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; visual mesh filename=/home/samaksh/biped_dev/RLstuff/Rocon-Biped-Genesis/urdf/me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
- link fix_leftfemur1_2: geometry collision mesh filename=/home/samaksh/biped_dev/RLstuff/Rocon-Biped-Genesis/urdf/me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; visual mesh filename=/home/samaksh/biped_dev/RLstuff/Rocon-Biped-Genesis/urdf/me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
- link fix_lefthip1motorbody: geometry collision mesh filename=/home/samaksh/biped_dev/RLstuff/Rocon-Biped-Genesis/urdf/me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; visual mesh filename=/home/samaksh/biped_dev/RLstuff/Rocon-Biped-Genesis/urdf/me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
- link fix_lefthip1towaist: geometry collision mesh filename=/home/samaksh/biped_dev/RLstuff/Rocon-Biped-Genesis/urdf/me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; visual mesh filename=/home/samaksh/biped_dev/RLstuff/Rocon-Biped-Genesis/urdf/me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
- link fix_leftlegtobaselink: geometry collision mesh filename=/home/samaksh/biped_dev/RLstuff/Rocon-Biped-Genesis/urdf/me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; visual mesh filename=/home/samaksh/biped_dev/RLstuff/Rocon-Biped-Genesis/urdf/me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
- link fix_lefttibia_1: mass 0.04 -> 0.048; geometry collision mesh filename=/home/samaksh/biped_dev/RLstuff/Rocon-Biped-Genesis/urdf/me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; visual mesh filename=/home/samaksh/biped_dev/RLstuff/Rocon-Biped-Genesis/urdf/me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
- link fix_lefttibia_2: geometry collision mesh filename=/home/samaksh/biped_dev/RLstuff/Rocon-Biped-Genesis/urdf/me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; visual mesh filename=/home/samaksh/biped_dev/RLstuff/Rocon-Biped-Genesis/urdf/me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
- link fix_lefttibia_3: geometry collision mesh filename=/home/samaksh/biped_dev/RLstuff/Rocon-Biped-Genesis/urdf/me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; visual mesh filename=/home/samaksh/biped_dev/RLstuff/Rocon-Biped-Genesis/urdf/me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
- link fix_lefttibia_4: geometry collision mesh filename=/home/samaksh/biped_dev/RLstuff/Rocon-Biped-Genesis/urdf/me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; visual mesh filename=/home/samaksh/biped_dev/RLstuff/Rocon-Biped-Genesis/urdf/me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
- link fix_lefttibia_5: geometry collision mesh filename=/home/samaksh/biped_dev/RLstuff/Rocon-Biped-Genesis/urdf/me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; visual mesh filename=/home/samaksh/biped_dev/RLstuff/Rocon-Biped-Genesis/urdf/me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
- link fix_lefttibia_6: geometry collision mesh filename=/home/samaksh/biped_dev/RLstuff/Rocon-Biped-Genesis/urdf/me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; visual mesh filename=/home/samaksh/biped_dev/RLstuff/Rocon-Biped-Genesis/urdf/me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
- link fix_right_femer1_2: geometry collision mesh filename=/home/samaksh/biped_dev/RLstuff/Rocon-Biped-Genesis/urdf/me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; visual mesh filename=/home/samaksh/biped_dev/RLstuff/Rocon-Biped-Genesis/urdf/me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
- link fix_right_femur2_2: geometry collision mesh filename=/home/samaksh/biped_dev/RLstuff/Rocon-Biped-Genesis/urdf/me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; visual mesh filename=/home/samaksh/biped_dev/RLstuff/Rocon-Biped-Genesis/urdf/me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
- link fix_right_femur2_3: geometry collision mesh filename=/home/samaksh/biped_dev/RLstuff/Rocon-Biped-Genesis/urdf/me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; visual mesh filename=/home/samaksh/biped_dev/RLstuff/Rocon-Biped-Genesis/urdf/me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
- link fix_right_hip1motorbody: geometry collision mesh filename=/home/samaksh/biped_dev/RLstuff/Rocon-Biped-Genesis/urdf/me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; visual mesh filename=/home/samaksh/biped_dev/RLstuff/Rocon-Biped-Genesis/urdf/me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
- link fix_rightfemer1_3: geometry collision mesh filename=/home/samaksh/biped_dev/RLstuff/Rocon-Biped-Genesis/urdf/me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; visual mesh filename=/home/samaksh/biped_dev/RLstuff/Rocon-Biped-Genesis/urdf/me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
- link fix_rightfemer1_4: geometry collision mesh filename=/home/samaksh/biped_dev/RLstuff/Rocon-Biped-Genesis/urdf/me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; visual mesh filename=/home/samaksh/biped_dev/RLstuff/Rocon-Biped-Genesis/urdf/me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
- link fix_righthip1towaist: geometry collision mesh filename=/home/samaksh/biped_dev/RLstuff/Rocon-Biped-Genesis/urdf/me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; visual mesh filename=/home/samaksh/biped_dev/RLstuff/Rocon-Biped-Genesis/urdf/me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
- link fix_rightlegtobaselink: geometry collision mesh filename=/home/samaksh/biped_dev/RLstuff/Rocon-Biped-Genesis/urdf/me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; visual mesh filename=/home/samaksh/biped_dev/RLstuff/Rocon-Biped-Genesis/urdf/me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
- link fix_righttibia_1: mass 0.04 -> 0.048; geometry collision mesh filename=/home/samaksh/biped_dev/RLstuff/Rocon-Biped-Genesis/urdf/me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; visual mesh filename=/home/samaksh/biped_dev/RLstuff/Rocon-Biped-Genesis/urdf/me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
- link fix_righttibia_2: geometry collision mesh filename=/home/samaksh/biped_dev/RLstuff/Rocon-Biped-Genesis/urdf/me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; visual mesh filename=/home/samaksh/biped_dev/RLstuff/Rocon-Biped-Genesis/urdf/me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
- link fix_righttibia_3: geometry collision mesh filename=/home/samaksh/biped_dev/RLstuff/Rocon-Biped-Genesis/urdf/me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; visual mesh filename=/home/samaksh/biped_dev/RLstuff/Rocon-Biped-Genesis/urdf/me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
- link fix_righttibia_4: geometry collision mesh filename=/home/samaksh/biped_dev/RLstuff/Rocon-Biped-Genesis/urdf/me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; visual mesh filename=/home/samaksh/biped_dev/RLstuff/Rocon-Biped-Genesis/urdf/me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
- link fix_righttibia_5: geometry collision mesh filename=/home/samaksh/biped_dev/RLstuff/Rocon-Biped-Genesis/urdf/me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; visual mesh filename=/home/samaksh/biped_dev/RLstuff/Rocon-Biped-Genesis/urdf/me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
- link fix_righttibia_6: geometry collision mesh filename=/home/samaksh/biped_dev/RLstuff/Rocon-Biped-Genesis/urdf/me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; visual mesh filename=/home/samaksh/biped_dev/RLstuff/Rocon-Biped-Genesis/urdf/me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
- link revolute_left_femur1_1: geometry collision mesh filename=/home/samaksh/biped_dev/RLstuff/Rocon-Biped-Genesis/urdf/me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; visual mesh filename=/home/samaksh/biped_dev/RLstuff/Rocon-Biped-Genesis/urdf/me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
- link revolute_left_femur2_1: geometry collision mesh filename=/home/samaksh/biped_dev/RLstuff/Rocon-Biped-Genesis/urdf/me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; visual mesh filename=/home/samaksh/biped_dev/RLstuff/Rocon-Biped-Genesis/urdf/me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
- link revolute_left_knee: geometry collision mesh filename=/home/samaksh/biped_dev/RLstuff/Rocon-Biped-Genesis/urdf/me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; visual mesh filename=/home/samaksh/biped_dev/RLstuff/Rocon-Biped-Genesis/urdf/me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
- link revolute_leftfoot: geometry collision mesh filename=/home/samaksh/biped_dev/RLstuff/Rocon-Biped-Genesis/urdf/me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; visual mesh filename=/home/samaksh/biped_dev/RLstuff/Rocon-Biped-Genesis/urdf/me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
- link revolute_right_femur2_1: geometry collision mesh filename=/home/samaksh/biped_dev/RLstuff/Rocon-Biped-Genesis/urdf/me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; visual mesh filename=/home/samaksh/biped_dev/RLstuff/Rocon-Biped-Genesis/urdf/me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
- link revolute_right_knee: geometry collision mesh filename=/home/samaksh/biped_dev/RLstuff/Rocon-Biped-Genesis/urdf/me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; visual mesh filename=/home/samaksh/biped_dev/RLstuff/Rocon-Biped-Genesis/urdf/me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
- link revolute_rightfemer1_1: geometry collision mesh filename=/home/samaksh/biped_dev/RLstuff/Rocon-Biped-Genesis/urdf/me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; visual mesh filename=/home/samaksh/biped_dev/RLstuff/Rocon-Biped-Genesis/urdf/me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
- link revolute_rightfoot: geometry collision mesh filename=/home/samaksh/biped_dev/RLstuff/Rocon-Biped-Genesis/urdf/me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; visual mesh filename=/home/samaksh/biped_dev/RLstuff/Rocon-Biped-Genesis/urdf/me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
Joints:
- removed joint base_joint
- removed joint cfpipe1tobaselink
- removed joint cfpipe2tobaselink
- removed joint torso
- removed joint torsolink1
- removed joint torsolink2
- removed joint torsolink3
- removed joint torsotobaselink
- removed joint torsotobaselink1
- removed joint torsoweight
- added joint fixedcfpipe1: type continuous, parent base_link, child cfpipebase1, origin xyz=0 0 0 rpy=3.14159265358979 1.5707963267949 0, axis 0 1 0
- added joint fixedcfpipe2: type continuous, parent base_link, child cfpipebase2, origin xyz=0.01375 0 0.00925 rpy=3.14159265358979 1.5707963267949 0, axis 0 1 0
- added joint left_sensor: type fixed, parent fixed_left_sensor_motor, child revolute_left_sensorstick, origin xyz=-0.024 0.0440346964193402 0.03655 rpy=0 0 -1.57079632679489, axis 0 0 0
- added joint left_sensor_motor: type fixed, parent revolute_leftfoot, child fixed_left_sensor_motor, origin xyz=0 0 0 rpy=0 0 0, axis 0 0 0
- added joint right_sensor: type revolute, parent fixed_right_sensor_motor, child revolute_right_sensorstick, origin xyz=-0.0440346964193401 -0.023999999999993 -0.0365499999999997 rpy=-3.14159265358979 0 3.14159265358979, axis 0 0 -1, limit lower=0 upper=0 effort=0 velocity=0
- added joint right_sensor_motor: type fixed, parent revolute_rightfoot, child fixed_right_sensor_motor, origin xyz=0 0 0 rpy=0 0 0, axis 0 0 0
- joint left_ankle: limit lower=-1.732 upper=1.732 effort=1 velocity=2 -> lower=-1.732 upper=1.732 effort=1.5 velocity=10
- joint left_hip1: limit lower=0 upper=0.3 effort=1.5 velocity=2 -> lower=-1.732 upper=1.732 effort=3.7 velocity=10
- joint left_hip2: limit lower=-1.732 upper=1.732 effort=1.5 velocity=2 -> lower=-1.732 upper=1.732 effort=3.7 velocity=10
- joint left_knee: axis 0 0 1 -> 0 0 -1; limit lower=-2 upper=2 effort=1.5 velocity=2 -> lower=-2 upper=2 effort=5 velocity=10
- joint right_ankle: axis 0 0 -1 -> 0 0 1; limit lower=-1.732 upper=1.732 effort=1 velocity=2 -> lower=-1.732 upper=1.732 effort=1.5 velocity=10
- joint right_hip1: limit lower=-0.3 upper=0 effort=1.5 velocity=2 -> lower=-1.732 upper=1.732 effort=3.7 velocity=10
- joint right_hip2: axis 0 0 -1 -> 0 0 1; limit lower=-1.732 upper=1.732 effort=1.5 velocity=2 -> lower=-1.732 upper=1.732 effort=3.7 velocity=10
- joint right_knee: axis 0 0 -1 -> 0 0 1; limit lower=-2 upper=2 effort=1.5 velocity=2 -> lower=-2 upper=2 effort=5 velocity=10

Commit message: inotial commit of setup

File: urdf/biped_v4.urdf (robot description, URDF)
Before this commit: robot biped_v4, 47 links, 46 joints
Links:
- removed link fix_torsolink1
- removed link fix_torsolink2
- removed link fix_torsolink3
- removed link fix_torsoweight
- removed link servo1
Joints:
- removed joint torso
- removed joint torsolink1
- removed joint torsolink2
- removed joint torsolink3
- removed joint torsoweight
- joint left_ankle: limit lower=-1.732 upper=1.732 effort=1 velocity=2 -> lower=-1.732 upper=1.732 effort=1.5 velocity=10
- joint left_hip1: limit lower=0 upper=0.3 effort=1.5 velocity=2 -> lower=-1.732 upper=1.732 effort=3.7 velocity=10
- joint left_hip2: limit lower=-1.732 upper=1.732 effort=1.5 velocity=2 -> lower=-1.732 upper=1.732 effort=3.7 velocity=10
- joint left_knee: limit lower=-2 upper=2 effort=1.5 velocity=2 -> lower=-2 upper=2 effort=5 velocity=10
- joint right_ankle: limit lower=-1.732 upper=1.732 effort=1 velocity=2 -> lower=-1.732 upper=1.732 effort=1.5 velocity=10
- joint right_hip1: limit lower=-0.3 upper=0 effort=1.5 velocity=2 -> lower=-1.732 upper=1.732 effort=3.7 velocity=10
- joint right_hip2: limit lower=-1.732 upper=1.732 effort=1.5 velocity=2 -> lower=-1.732 upper=1.732 effort=3.7 velocity=10
- joint right_knee: limit lower=-2 upper=2 effort=1.5 velocity=2 -> lower=-2 upper=2 effort=5 velocity=10

Commit message: reward switch options and urdf effort and vel limits

File: urdf/biped_v4.urdf (robot description, URDF)
Before this commit: robot biped_v4, 42 links, 41 joints
Joints:
- joint left_ankle: limit lower=-1.732 upper=1.732 effort=1.5 velocity=10 -> lower=-1.732 upper=1.732 effort=1.5 velocity=3
- joint left_hip1: limit lower=-1.732 upper=1.732 effort=3.7 velocity=10 -> lower=-1.732 upper=1.732 effort=1.5 velocity=3
- joint left_hip2: limit lower=-1.732 upper=1.732 effort=3.7 velocity=10 -> lower=-1.732 upper=1.732 effort=2 velocity=4.2
- joint left_knee: limit lower=-2 upper=2 effort=5 velocity=10 -> lower=-2 upper=2 effort=1.5 velocity=3
- joint right_ankle: limit lower=-1.732 upper=1.732 effort=1.5 velocity=10 -> lower=-1.732 upper=1.732 effort=1.5 velocity=3
- joint right_hip1: limit lower=-1.732 upper=1.732 effort=3.7 velocity=10 -> lower=-1.732 upper=1.732 effort=1.5 velocity=3
- joint right_hip2: limit lower=-1.732 upper=1.732 effort=3.7 velocity=10 -> lower=-1.732 upper=1.732 effort=2 velocity=4.2
- joint right_knee: limit lower=-2 upper=2 effort=5 velocity=10 -> lower=-2 upper=2 effort=1.5 velocity=3

Commit message: urdf edits and low height episode termination

File: urdf/biped_v4.urdf (robot description, URDF)
Before this commit: robot biped_v4, 42 links, 41 joints
Joints:
- joint left_ankle: limit lower=-1.732 upper=1.732 effort=1.5 velocity=3 -> lower=-1.732 upper=1.732 effort=5 velocity=3
- joint left_hip1: limit lower=-1.732 upper=1.732 effort=1.5 velocity=3 -> lower=-1.732 upper=1.732 effort=5 velocity=3
- joint left_hip2: limit lower=-1.732 upper=1.732 effort=2 velocity=4.2 -> lower=-1.732 upper=1.732 effort=5 velocity=4.2
- joint left_knee: limit lower=-2 upper=2 effort=1.5 velocity=3 -> lower=-2 upper=2 effort=5 velocity=3
- joint right_ankle: limit lower=-1.732 upper=1.732 effort=1.5 velocity=3 -> lower=-1.732 upper=1.732 effort=5 velocity=3
- joint right_hip1: limit lower=-1.732 upper=1.732 effort=1.5 velocity=3 -> lower=-1.732 upper=1.732 effort=5 velocity=3
- joint right_hip2: limit lower=-1.732 upper=1.732 effort=2 velocity=4.2 -> lower=-1.732 upper=1.732 effort=5 velocity=4.2
- joint right_knee: limit lower=-2 upper=2 effort=1.5 velocity=3 -> lower=-2 upper=2 effort=5 velocity=3

Commit message: just urdf update

File: urdf/biped_v4.urdf (robot description, URDF)
Before this commit: robot biped_v4, 47 links, 46 joints
Joints:
- joint left_ankle: limit lower=-1.732 upper=1.732 effort=1 velocity=2 -> lower=-1.732 upper=1.732 effort=5 velocity=5
- joint left_hip1: limit lower=0 upper=0.3 effort=1.5 velocity=2 -> lower=0 upper=0.3 effort=5 velocity=4
- joint left_hip2: limit lower=-1.732 upper=1.732 effort=1.5 velocity=2 -> lower=-1.732 upper=1.732 effort=5 velocity=5
- joint left_knee: limit lower=-2 upper=2 effort=1.5 velocity=2 -> lower=-2 upper=2 effort=5 velocity=5
- joint right_ankle: limit lower=-1.732 upper=1.732 effort=1 velocity=2 -> lower=-1.732 upper=1.732 effort=5 velocity=5
- joint right_hip1: limit lower=-0.3 upper=0 effort=1.5 velocity=2 -> lower=-0.3 upper=0 effort=5 velocity=5
- joint right_hip2: limit lower=-1.732 upper=1.732 effort=1.5 velocity=2 -> lower=-1.732 upper=1.732 effort=5 velocity=5
- joint right_knee: limit lower=-2 upper=2 effort=1.5 velocity=2 -> lower=-2 upper=2 effort=5 velocity=5
- joint torso: limit lower=-1.0 upper=1.0 effort=1.8 velocity=1.8 -> lower=-1.0 upper=1.0 effort=5 velocity=5
