Commit message: changed URDF

File: urdf/biped_v4.urdf (robot description, URDF)
Before this commit: robot biped_v4, 47 links, 46 joints
Links:
- removed link world
- added link fixed_left_sensor_motor, mass 0.02; collision mesh filename=/home/samaksh/biped_dev/RLstuff/Rocon-Biped-Genesis/urdf/me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; visual mesh filename=/home/samaksh/biped_dev/RLstuff/Rocon-Biped-Genesis/urdf/me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
- added link fixed_right_sensor_motor, mass 0.02; collision mesh filename=/home/samaksh/biped_dev/RLstuff/Rocon-Biped-Genesis/urdf/me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; visual mesh filename=/home/samaksh/biped_dev/RLstuff/Rocon-Biped-Genesis/urdf/me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
- added link revolute_left_sensorstick, mass 0.003; collision mesh filename=/home/samaksh/biped_dev/RLstuff/Rocon-Biped-Genesis/urdf/me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; visual mesh filename=/home/samaksh/biped_dev/RLstuff/Rocon-Biped-Genesis/urdf/me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
- added link revolute_right_sensorstick, mass 0.003; collision mesh filename=/home/samaksh/biped_dev/RLstuff/Rocon-Biped-Genesis/urdf/me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; visual mesh filename=/home/samaksh/biped_dev/RLstuff/Rocon-Biped-Genesis/urdf/me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
- link base_link: geometry collision mesh filename=/home/samaksh/biped_dev/RLstuff/Rocon-Biped-Genesis/urdf/me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; visual mesh filename=/home/samaksh/biped_dev/RLstuff/Rocon-Biped-Genesis/urdf/me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
- link fix_cfpipe1tobaselink: geometry collision mesh filename=/home/samaksh/biped_dev/RLstuff/Rocon-Biped-Genesis/urdf/me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; visual mesh filename=/home/samaksh/biped_dev/RLstuff/Rocon-Biped-Genesis/urdf/me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
- link fix_cfpipe2tobaselink: geometry collision mesh filename=/home/samaksh/biped_dev/RLstuff/Rocon-Biped-Genesis/urdf/me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; visual mesh filename=/home/samaksh/biped_dev/RLstuff/Rocon-Biped-Genesis/urdf/me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
- link fix_femur1_3: geometry collision mesh filename=/home/samaksh/biped_dev/RLstuff/Rocon-Biped-Genesis/urdf/me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; visual mesh filename=/home/samaksh/biped_dev/RLstuff/Rocon-Biped-Genesis/urdf/me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
- link fix_femur1_4: geometry collision mesh filename=/home/samaksh/biped_dev/RLstuff/Rocon-Biped-Genesis/urdf/me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; visual mesh filename=/home/samaksh/biped_dev/RLstuff/Rocon-Biped-Genesis/urdf/me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
- link fix_left_femur2_2: geometry collision mesh filename=/home/samaksh/biped_dev/RLstuff/Rocon-Biped-Genesis/urdf/me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; visual mesh filename=/home/samaksh/biped_dev/RLstuff/Rocon-Biped-Genesis/urdf/me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
- link fix_left_femur2_3: geometry collision mesh filename=/home/samaksh/biped_dev/RLstuff/Rocon-Biped-Genesis/urdf/me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; visual mesh filename=/home/samaksh/biped_dev/RLstuff/Rocon-Biped-Genesis/urdf/me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
- link fix_leftfemur1_2: geometry collision mesh filename=/home/samaksh/biped_dev/RLstuff/Rocon-Biped-Genesis/urdf/me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; visual mesh filename=/home/samaksh/biped_dev/RLstuff/Rocon-Biped-Genesis/urdf/me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
- link fix_lefthip1motorbody: geometry collision mesh filename=/home/samaksh/biped_dev/RLstuff/Rocon-Biped-Genesis/urdf/me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; visual mesh filename=/home/samaksh/biped_dev/RLstuff/Rocon-Biped-Genesis/urdf/me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
- link fix_lefthip1towaist: geometry collision mesh filename=/home/samaksh/biped_dev/RLstuff/Rocon-Biped-Genesis/urdf/me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; visual mesh filename=/home/samaksh/biped_dev/RLstuff/Rocon-Biped-Genesis/urdf/me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
- link fix_leftlegtobaselink: geometry collision mesh filename=/home/samaksh/biped_dev/RLstuff/Rocon-Biped-Genesis/urdf/me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; visual mesh filename=/home/samaksh/biped_dev/RLstuff/Rocon-Biped-Genesis/urdf/me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
- link fix_lefttibia_1: mass 0.04 -> 0.048; geometry collision mesh filename=/home/samaksh/biped_dev/RLstuff/Rocon-Biped-Genesis/urdf/me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; visual mesh filename=/home/samaksh/biped_dev/RLstuff/Rocon-Biped-Genesis/urdf/me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
- link fix_lefttibia_2: geometry collision mesh filename=/home/samaksh/biped_dev/RLstuff/Rocon-Biped-Genesis/urdf/me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; visual mesh filename=/home/samaksh/biped_dev/RLstuff/Rocon-Biped-Genesis/urdf/me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
- link fix_lefttibia_3: geometry collision mesh filename=/home/samaksh/biped_dev/RLstuff/Rocon-Biped-Genesis/urdf/me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; visual mesh filename=/home/samaksh/biped_dev/RLstuff/Rocon-Biped-Genesis/urdf/me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
- link fix_lefttibia_4: geometry collision mesh filename=/home/samaksh/biped_dev/RLstuff/Rocon-Biped-Genesis/urdf/me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; visual mesh filename=/home/samaksh/biped_dev/RLstuff/Rocon-Biped-Genesis/urdf/me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
- link fix_lefttibia_5: geometry collision mesh filename=/home/samaksh/biped_dev/RLstuff/Rocon-Biped-Genesis/urdf/me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; visual mesh filename=/home/samaksh/biped_dev/RLstuff/Rocon-Biped-Genesis/urdf/me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
- link fix_lefttibia_6: geometry collision mesh filename=/home/samaksh/biped_dev/RLstuff/Rocon-Biped-Genesis/urdf/me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; visual mesh filename=/home/samaksh/biped_dev/RLstuff/Rocon-Biped-Genesis/urdf/me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
- link fix_right_femer1_2: geometry collision mesh filename=/home/samaksh/biped_dev/RLstuff/Rocon-Biped-Genesis/urdf/me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; visual mesh filename=/home/samaksh/biped_dev/RLstuff/Rocon-Biped-Genesis/urdf/me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
- link fix_right_femur2_2: geometry collision mesh filename=/home/samaksh/biped_dev/RLstuff/Rocon-Biped-Genesis/urdf/me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; visual mesh filename=/home/samaksh/biped_dev/RLstuff/Rocon-Biped-Genesis/urdf/me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
- link fix_right_femur2_3: geometry collision mesh filename=/home/samaksh/biped_dev/RLstuff/Rocon-Biped-Genesis/urdf/me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; visual mesh filename=/home/samaksh/biped_dev/RLstuff/Rocon-Biped-Genesis/urdf/me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
- link fix_right_hip1motorbody: geometry collision mesh filename=/home/samaksh/biped_dev/RLstuff/Rocon-Biped-Genesis/urdf/me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; visual mesh filename=/home/samaksh/biped_dev/RLstuff/Rocon-Biped-Genesis/urdf/me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
- link fix_rightfemer1_3: geometry collision mesh filename=/home/samaksh/biped_dev/RLstuff/Rocon-Biped-Genesis/urdf/me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; visual mesh filename=/home/samaksh/biped_dev/RLstuff/Rocon-Biped-Genesis/urdf/me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
- link fix_rightfemer1_4: geometry collision mesh filename=/home/samaksh/biped_dev/RLstuff/Rocon-Biped-Genesis/urdf/me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; visual mesh filename=/home/samaksh/biped_dev/RLstuff/Rocon-Biped-Genesis/urdf/me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
- link fix_righthip1towaist: geometry collision mesh filename=/home/samaksh/biped_dev/RLstuff/Rocon-Biped-Genesis/urdf/me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; visual mesh filename=/home/samaksh/biped_dev/RLstuff/Rocon-Biped-Genesis/urdf/me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
- link fix_rightlegtobaselink: geometry collision mesh filename=/home/samaksh/biped_dev/RLstuff/Rocon-Biped-Genesis/urdf/me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; visual mesh filename=/home/samaksh/biped_dev/RLstuff/Rocon-Biped-Genesis/urdf/me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
- link fix_righttibia_1: mass 0.04 -> 0.048; geometry collision mesh filename=/home/samaksh/biped_dev/RLstuff/Rocon-Biped-Genesis/urdf/me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; visual mesh filename=/home/samaksh/biped_dev/RLstuff/Rocon-Biped-Genesis/urdf/me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
- link fix_righttibia_2: geometry collision mesh filename=/home/samaksh/biped_dev/RLstuff/Rocon-Biped-Genesis/urdf/me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; visual mesh filename=/home/samaksh/biped_dev/RLstuff/Rocon-Biped-Genesis/urdf/me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
- link fix_righttibia_3: geometry collision mesh filename=/home/samaksh/biped_dev/RLstuff/Rocon-Biped-Genesis/urdf/me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; visual mesh filename=/home/samaksh/biped_dev/RLstuff/Rocon-Biped-Genesis/urdf/me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
- link fix_righttibia_4: geometry collision mesh filename=/home/samaksh/biped_dev/RLstuff/Rocon-Biped-Genesis/urdf/me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; visual mesh filename=/home/samaksh/biped_dev/RLstuff/Rocon-Biped-Genesis/urdf/me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
- link fix_righttibia_5: geometry collision mesh filename=/home/samaksh/biped_dev/RLstuff/Rocon-Biped-Genesis/urdf/me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; visual mesh filename=/home/samaksh/biped_dev/RLstuff/Rocon-Biped-Genesis/urdf/me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
- link fix_righttibia_6: geometry collision mesh filename=/home/samaksh/biped_dev/RLstuff/Rocon-Biped-Genesis/urdf/me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; visual mesh filename=/home/samaksh/biped_dev/RLstuff/Rocon-Biped-Genesis/urdf/me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
- link fix_torsolink1: mass 0.01 -> 0.009726; geometry collision mesh filename=/home/samaksh/biped_dev/RLstuff/Rocon-Biped-Genesis/urdf/me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; visual mesh filename=/home/samaksh/biped_dev/RLstuff/Rocon-Biped-Genesis/urdf/me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
- link fix_torsolink2: geometry collision mesh filename=/home/samaksh/biped_dev/RLstuff/Rocon-Biped-Genesis/urdf/me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; visual mesh filename=/home/samaksh/biped_dev/RLstuff/Rocon-Biped-Genesis/urdf/me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
- link fix_torsolink3: mass 0.006 -> 0.006125; geometry collision mesh filename=/home/samaksh/biped_dev/RLstuff/Rocon-Biped-Genesis/urdf/me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; visual mesh filename=/home/samaksh/biped_dev/RLstuff/Rocon-Biped-Genesis/urdf/me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
- link fix_torsotobaselink1: geometry collision mesh filename=/home/samaksh/biped_dev/RLstuff/Rocon-Biped-Genesis/urdf/me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; visual mesh filename=/home/samaksh/biped_dev/RLstuff/Rocon-Biped-Genesis/urdf/me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
- link fix_torsotobaselink2: geometry collision mesh filename=/home/samaksh/biped_dev/RLstuff/Rocon-Biped-Genesis/urdf/me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; visual mesh filename=/home/samaksh/biped_dev/RLstuff/Rocon-Biped-Genesis/urdf/me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
- link fix_torsoweight: geometry collision mesh filename=/home/samaksh/biped_dev/RLstuff/Rocon-Biped-Genesis/urdf/me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; visual mesh filename=/home/samaksh/biped_dev/RLstuff/Rocon-Biped-Genesis/urdf/me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
- link revolute_left_femur1_1: geometry collision mesh filename=/home/samaksh/biped_dev/RLstuff/Rocon-Biped-Genesis/urdf/me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; visual mesh filename=/home/samaksh/biped_dev/RLstuff/Rocon-Biped-Genesis/urdf/me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
- link revolute_left_femur2_1: geometry collision mesh filename=/home/samaksh/biped_dev/RLstuff/Rocon-Biped-Genesis/urdf/me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; visual mesh filename=/home/samaksh/biped_dev/RLstuff/Rocon-Biped-Genesis/urdf/me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
- link revolute_left_knee: geometry collision mesh filename=/home/samaksh/biped_dev/RLstuff/Rocon-Biped-Genesis/urdf/me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; visual mesh filename=/home/samaksh/biped_dev/RLstuff/Rocon-Biped-Genesis/urdf/me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
- link revolute_leftfoot: geometry collision mesh filename=/home/samaksh/biped_dev/RLstuff/Rocon-Biped-Genesis/urdf/me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; visual mesh filename=/home/samaksh/biped_dev/RLstuff/Rocon-Biped-Genesis/urdf/me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
- link revolute_right_femur2_1: geometry collision mesh filename=/home/samaksh/biped_dev/RLstuff/Rocon-Biped-Genesis/urdf/me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; visual mesh filename=/home/samaksh/biped_dev/RLstuff/Rocon-Biped-Genesis/urdf/me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
- link revolute_right_knee: geometry collision mesh filename=/home/samaksh/biped_dev/RLstuff/Rocon-Biped-Genesis/urdf/me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; visual mesh filename=/home/samaksh/biped_dev/RLstuff/Rocon-Biped-Genesis/urdf/me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
- link revolute_rightfemer1_1: geometry collision mesh filename=/home/samaksh/biped_dev/RLstuff/Rocon-Biped-Genesis/urdf/me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; visual mesh filename=/home/samaksh/biped_dev/RLstuff/Rocon-Biped-Genesis/urdf/me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
- link revolute_rightfoot: geometry collision mesh filename=/home/samaksh/biped_dev/RLstuff/Rocon-Biped-Genesis/urdf/me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; visual mesh filename=/home/samaksh/biped_dev/RLstuff/Rocon-Biped-Genesis/urdf/me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
- link servo1: mass 0.165 -> 0.048; geometry collision mesh filename=/home/samaksh/biped_dev/RLstuff/Rocon-Biped-Genesis/urdf/me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; visual mesh filename=/home/samaksh/biped_dev/RLstuff/Rocon-Biped-Genesis/urdf/me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
Joints:
- removed joint base_joint
- removed joint torso
- added joint left_sensor: type fixed, parent fixed_left_sensor_motor, child revolute_left_sensorstick, origin xyz=-0.024 0.044035 0.03655 rpy=0 0 -1.5708, axis 0 0 0
- added joint left_sensor_motor: type fixed, parent revolute_leftfoot, child fixed_left_sensor_motor, origin xyz=0 0 0 rpy=0 0 0, axis 0 0 0
- added joint revolute_torso: type revolute, parent fix_torsotobaselink1, child servo1, origin xyz=0 0.0298000000000001 0.0422500000000002 rpy=1.57079632679489 0 1.5707963267949, axis 1 0 0, limit lower=-1.732 upper=1.732 effort=13 velocity=10
- added joint right_sensor: type fixed, parent fixed_right_sensor_motor, child revolute_right_sensorstick, origin xyz=0 0 0 rpy=0 0 0, axis 0 0 1, limit lower=0 upper=0 effort=0 velocity=0
- added joint right_sensor_motor: type fixed, parent revolute_rightfoot, child fixed_right_sensor_motor, origin xyz=0 0 0 rpy=0 0 0, axis 0 0 0
- joint cfpipe1tobaselink: type fixed -> continuous
- joint left_ankle: limit lower=-1.732 upper=1.732 effort=5 velocity=5 -> lower=-1.732 upper=1.732 effort=1.5 velocity=10; origin xyz=0 -0.181000000000001 0.00250000000000145 rpy=0 0 1.57079632679489 -> xyz=0 -0.156 0.0025 rpy=0 0 1.5708
- joint left_hip1: limit lower=0 upper=0.3 effort=5 velocity=4 -> lower=-1.732 upper=1.732 effort=3.7 velocity=10; origin xyz=-0.0234 -0.09425 -0.024125 rpy=0 1.5707963267949 0 -> xyz=-0.0234 -0.08425 -0.024125 rpy=0 1.5708 0
- joint left_hip2: limit lower=-1.732 upper=1.732 effort=5 velocity=5 -> lower=-1.732 upper=1.732 effort=3.7 velocity=10; origin xyz=0.048875 -0.0234 0.00939999999999994 rpy=1.5707963267949 -1.5707963267949 0 -> xyz=0.048875 -0.0234 0.0094 rpy=1.5708 -1.5708 0
- joint left_knee: axis 0 0 1 -> 0 0 -1; limit lower=-2 upper=2 effort=5 velocity=5 -> lower=-2 upper=2 effort=5 velocity=10; origin xyz=0 -0.162 0 rpy=-3.14159265358979 0 -3.14159265358979 -> xyz=0 -0.137 0 rpy=-3.1416 0 -3.1416
- joint lefthip1motorbody: origin xyz=-0.0234 -0.09425 -0.024125 rpy=0 1.5707963267949 0 -> xyz=-0.0234 -0.08425 -0.024125 rpy=0 1.5708 0
- joint right_ankle: axis 0 0 -1 -> 0 0 1; limit lower=-1.732 upper=1.732 effort=5 velocity=5 -> lower=-1.732 upper=1.732 effort=1.5 velocity=10; origin xyz=0 -0.181000000000001 -0.00250000000000579 rpy=0 0 0 -> xyz=0 -0.156 -0.0025 rpy=0 0 0
- joint right_hip1: limit lower=-0.3 upper=0 effort=5 velocity=5 -> lower=-1.732 upper=1.732 effort=3.7 velocity=10; origin xyz=-0.0234 0.09425 -0.024125 rpy=1.5707963267949 0 1.5707963267949 -> xyz=-0.0234 0.08425 -0.024125 rpy=1.5708 0 1.5708
- joint right_hip2: axis 0 0 -1 -> 0 0 1; limit lower=-1.732 upper=1.732 effort=5 velocity=5 -> lower=-1.732 upper=1.732 effort=3.7 velocity=10; origin xyz=0.0233999999999999 -0.048875 0.00940000000000001 rpy=0 1.5707963267949 0 -> xyz=0.0234 -0.048875 0.0094 rpy=0 1.5708 0
- joint right_knee: axis 0 0 -1 -> 0 0 1; limit lower=-2 upper=2 effort=5 velocity=5 -> lower=-2 upper=2 effort=5 velocity=10; origin xyz=0 -0.162000000000005 0 rpy=0 0 0 -> xyz=0 -0.137 0 rpy=0 0 0
