Commit message: adjusted torsoless

File: urdf/biped_v4.urdf (robot description, URDF)
Before this commit: robot biped_v4, 43 links, 42 joints
Links:
- removed link cfpipebase1
- removed link cfpipebase2
- removed link revolute_left_sensorstick
- removed link revolute_right_sensorstick
- added link fix_cfpipe1tobaselink, mass 0.007; collision mesh filename=/home/samaksh/biped_dev/RLstuff/Biped_RL/urdf/meshes/fix_cf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; visual mesh filename=/home/samaksh/biped_dev/RLstuff/Biped_RL/urdf/meshes/fix_cf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
- added link fix_cfpipe2tobaselink, mass 0.007; collision mesh filename=/home/samaksh/biped_dev/RLstuff/Biped_RL/urdf/meshes/fix_cf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; visual mesh filename=/home/samaksh/biped_dev/RLstuff/Biped_RL/urdf/meshes/fix_cf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
- added link fix_torsotobaselink1, mass 0.02; collision mesh filename=/home/samaksh/biped_dev/RLstuff/Biped_RL/urdf/meshes/fix_to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; visual mesh filename=/home/samaksh/biped_dev/RLstuff/Biped_RL/urdf/meshes/fix_to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
- link base_link: geometry collision mesh filename=/home/samaksh/biped_dev/RLstuff/Biped_RL/urdf/meshes/base_l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; visual mesh filename=/home/samaksh/biped_dev/RLstuff/Biped_RL/urdf/meshes/base_l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
- link fix_femur1_3: geometry collision mesh filename=/home/samaksh/biped_dev/RLstuff/Biped_RL/urdf/meshes/fix_fe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; visual mesh filename=/home/samaksh/biped_dev/RLstuff/Biped_RL/urdf/meshes/fix_fe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
- link fix_femur1_4: geometry collision mesh filename=/home/samaksh/biped_dev/RLstuff/Biped_RL/urdf/meshes/fix_fe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; visual mesh filename=/home/samaksh/biped_dev/RLstuff/Biped_RL/urdf/meshes/fix_fe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
- link fix_left_femur2_2: geometry collision mesh filename=/home/samaksh/biped_dev/RLstuff/Biped_RL/urdf/meshes/fix_le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; visual mesh filename=/home/samaksh/biped_dev/RLstuff/Biped_RL/urdf/meshes/fix_le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
- link fix_left_femur2_3: geometry collision mesh filename=/home/samaksh/biped_dev/RLstuff/Biped_RL/urdf/meshes/fix_le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; visual mesh filename=/home/samaksh/biped_dev/RLstuff/Biped_RL/urdf/meshes/fix_le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
- link fix_leftfemur1_2: geometry collision mesh filename=/home/samaksh/biped_dev/RLstuff/Biped_RL/urdf/meshes/fix_le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; visual mesh filename=/home/samaksh/biped_dev/RLstuff/Biped_RL/urdf/meshes/fix_le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
- link fix_lefthip1motorbody: geometry collision mesh filename=/home/samaksh/biped_dev/RLstuff/Biped_RL/urdf/meshes/fix_le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; visual mesh filename=/home/samaksh/biped_dev/RLstuff/Biped_RL/urdf/meshes/fix_le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
- link fix_lefthip1towaist: geometry collision mesh filename=/home/samaksh/biped_dev/RLstuff/Biped_RL/urdf/meshes/fix_le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; visual mesh filename=/home/samaksh/biped_dev/RLstuff/Biped_RL/urdf/meshes/fix_le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
- link fix_leftlegtobaselink: geometry collision mesh filename=/home/samaksh/biped_dev/RLstuff/Biped_RL/urdf/meshes/fix_le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; visual mesh filename=/home/samaksh/biped_dev/RLstuff/Biped_RL/urdf/meshes/fix_le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
- link fix_lefttibia_1: geometry collision mesh filename=/home/samaksh/biped_dev/RLstuff/Biped_RL/urdf/meshes/fix_le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; visual mesh filename=/home/samaksh/biped_dev/RLstuff/Biped_RL/urdf/meshes/fix_le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
- link fix_lefttibia_2: geometry collision mesh filename=/home/samaksh/biped_dev/RLstuff/Biped_RL/urdf/meshes/fix_le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; visual mesh filename=/home/samaksh/biped_dev/RLstuff/Biped_RL/urdf/meshes/fix_le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
- link fix_lefttibia_3: geometry collision mesh filename=/home/samaksh/biped_dev/RLstuff/Biped_RL/urdf/meshes/fix_le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; visual mesh filename=/home/samaksh/biped_dev/RLstuff/Biped_RL/urdf/meshes/fix_le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
- link fix_lefttibia_4: geometry collision mesh filename=/home/samaksh/biped_dev/RLstuff/Biped_RL/urdf/meshes/fix_le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; visual mesh filename=/home/samaksh/biped_dev/RLstuff/Biped_RL/urdf/meshes/fix_le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
- link fix_lefttibia_5: geometry collision mesh filename=/home/samaksh/biped_dev/RLstuff/Biped_RL/urdf/meshes/fix_le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; visual mesh filename=/home/samaksh/biped_dev/RLstuff/Biped_RL/urdf/meshes/fix_le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
- link fix_lefttibia_6: geometry collision mesh filename=/home/samaksh/biped_dev/RLstuff/Biped_RL/urdf/meshes/fix_le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; visual mesh filename=/home/samaksh/biped_dev/RLstuff/Biped_RL/urdf/meshes/fix_le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
- link fix_right_femer1_2: geometry collision mesh filename=/home/samaksh/biped_dev/RLstuff/Biped_RL/urdf/meshes/fix_ri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; visual mesh filename=/home/samaksh/biped_dev/RLstuff/Biped_RL/urdf/meshes/fix_ri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
- link fix_right_femur2_2: geometry collision mesh filename=/home/samaksh/biped_dev/RLstuff/Biped_RL/urdf/meshes/fix_ri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; visual mesh filename=/home/samaksh/biped_dev/RLstuff/Biped_RL/urdf/meshes/fix_ri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
- link fix_right_femur2_3: geometry collision mesh filename=/home/samaksh/biped_dev/RLstuff/Biped_RL/urdf/meshes/fix_ri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; visual mesh filename=/home/samaksh/biped_dev/RLstuff/Biped_RL/urdf/meshes/fix_ri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
- link fix_right_hip1motorbody: geometry collision mesh filename=/home/samaksh/biped_dev/RLstuff/Biped_RL/urdf/meshes/fix_ri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; visual mesh filename=/home/samaksh/biped_dev/RLstuff/Biped_RL/urdf/meshes/fix_ri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
- link fix_rightfemer1_3: geometry collision mesh filename=/home/samaksh/biped_dev/RLstuff/Biped_RL/urdf/meshes/fix_ri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; visual mesh filename=/home/samaksh/biped_dev/RLstuff/Biped_RL/urdf/meshes/fix_ri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
- link fix_rightfemer1_4: geometry collision mesh filename=/home/samaksh/biped_dev/RLstuff/Biped_RL/urdf/meshes/fix_ri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; visual mesh filename=/home/samaksh/biped_dev/RLstuff/Biped_RL/urdf/meshes/fix_ri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
- link fix_righthip1towaist: geometry collision mesh filename=/home/samaksh/biped_dev/RLstuff/Biped_RL/urdf/meshes/fix_ri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; visual mesh filename=/home/samaksh/biped_dev/RLstuff/Biped_RL/urdf/meshes/fix_ri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
- link fix_rightlegtobaselink: geometry collision mesh filename=/home/samaksh/biped_dev/RLstuff/Biped_RL/urdf/meshes/fix_ri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; visual mesh filename=/home/samaksh/biped_dev/RLstuff/Biped_RL/urdf/meshes/fix_ri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
- link fix_righttibia_1: geometry collision mesh filename=/home/samaksh/biped_dev/RLstuff/Biped_RL/urdf/meshes/fix_ri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; visual mesh filename=/home/samaksh/biped_dev/RLstuff/Biped_RL/urdf/meshes/fix_ri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
- link fix_righttibia_2: geometry collision mesh filename=/home/samaksh/biped_dev/RLstuff/Biped_RL/urdf/meshes/fix_ri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; visual mesh filename=/home/samaksh/biped_dev/RLstuff/Biped_RL/urdf/meshes/fix_ri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
- link fix_righttibia_3: geometry collision mesh filename=/home/samaksh/biped_dev/RLstuff/Biped_RL/urdf/meshes/fix_ri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; visual mesh filename=/home/samaksh/biped_dev/RLstuff/Biped_RL/urdf/meshes/fix_ri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
- link fix_righttibia_4: geometry collision mesh filename=/home/samaksh/biped_dev/RLstuff/Biped_RL/urdf/meshes/fix_ri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; visual mesh filename=/home/samaksh/biped_dev/RLstuff/Biped_RL/urdf/meshes/fix_ri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
- link fix_righttibia_5: geometry collision mesh filename=/home/samaksh/biped_dev/RLstuff/Biped_RL/urdf/meshes/fix_ri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; visual mesh filename=/home/samaksh/biped_dev/RLstuff/Biped_RL/urdf/meshes/fix_ri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
- link fix_righttibia_6: geometry collision mesh filename=/home/samaksh/biped_dev/RLstuff/Biped_RL/urdf/meshes/fix_ri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; visual mesh filename=/home/samaksh/biped_dev/RLstuff/Biped_RL/urdf/meshes/fix_ri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
- link fixed_left_sensor_motor: geometry collision mesh filename=/home/samaksh/biped_dev/RLstuff/Biped_RL/urdf/meshes/fixed_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; visual mesh filename=/home/samaksh/biped_dev/RLstuff/Biped_RL/urdf/meshes/fixed_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
- link fixed_right_sensor_motor: geometry collision mesh filename=/home/samaksh/biped_dev/RLstuff/Biped_RL/urdf/meshes/fixed_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; visual mesh filename=/home/samaksh/biped_dev/RLstuff/Biped_RL/urdf/meshes/fixed_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
- link revolute_left_femur1_1: geometry collision mesh filename=/home/samaksh/biped_dev/RLstuff/Biped_RL/urdf/meshes/revolu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; visual mesh filename=/home/samaksh/biped_dev/RLstuff/Biped_RL/urdf/meshes/revolu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
- link revolute_left_femur2_1: geometry collision mesh filename=/home/samaksh/biped_dev/RLstuff/Biped_RL/urdf/meshes/revolu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; visual mesh filename=/home/samaksh/biped_dev/RLstuff/Biped_RL/urdf/meshes/revolu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
- link revolute_left_knee: geometry collision mesh filename=/home/samaksh/biped_dev/RLstuff/Biped_RL/urdf/meshes/revolu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; visual mesh filename=/home/samaksh/biped_dev/RLstuff/Biped_RL/urdf/meshes/revolu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
- link revolute_leftfoot: geometry collision mesh filename=/home/samaksh/biped_dev/RLstuff/Biped_RL/urdf/meshes/revolu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; visual mesh filename=/home/samaksh/biped_dev/RLstuff/Biped_RL/urdf/meshes/revolu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
- link revolute_right_femur2_1: geometry collision mesh filename=/home/samaksh/biped_dev/RLstuff/Biped_RL/urdf/meshes/revolu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; visual mesh filename=/home/samaksh/biped_dev/RLstuff/Biped_RL/urdf/meshes/revolu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
- link revolute_right_knee: geometry collision mesh filename=/home/samaksh/biped_dev/RLstuff/Biped_RL/urdf/meshes/revolu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; visual mesh filename=/home/samaksh/biped_dev/RLstuff/Biped_RL/urdf/meshes/revolu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
- link revolute_rightfemer1_1: geometry collision mesh filename=/home/samaksh/biped_dev/RLstuff/Biped_RL/urdf/meshes/revolu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; visual mesh filename=/home/samaksh/biped_dev/RLstuff/Biped_RL/urdf/meshes/revolu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
- link revolute_rightfoot: geometry collision mesh filename=/home/samaksh/biped_dev/RLstuff/Biped_RL/urdf/meshes/revolu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; visual mesh filename=/home/samaksh/biped_dev/RLstuff/Biped_RL/urdf/meshes/revolu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
Joints:
- removed joint fixedcfpipe1
- removed joint fixedcfpipe2
- removed joint left_sensor
- removed joint right_sensor
- added joint cfpipe1tobaselink: type fixed, parent base_link, child fix_cfpipe1tobaselink, origin xyz=0 0 0 rpy=0 0 0
- added joint cfpipe2tobaselink: type fixed, parent base_link, child fix_cfpipe2tobaselink, origin xyz=0 0 0 rpy=0 0 0, axis 0 0 0
- added joint torsotobaselink1: type fixed, parent base_link, child fix_torsotobaselink1, origin xyz=0 0 0 rpy=0 0 0, axis 0 0 0
- joint left_ankle: origin xyz=0 -0.181000000000001 0.00250000000000145 rpy=0 0 1.57079632679489 -> xyz=0 -0.156 0.0025 rpy=0 0 1.5708
- joint left_hip1: origin xyz=-0.0234 -0.09425 -0.024125 rpy=0 1.5707963267949 0 -> xyz=-0.0234 -0.08425 -0.024125 rpy=0 1.5708 0
- joint left_hip2: origin xyz=0.048875 -0.0234 0.00939999999999994 rpy=1.5707963267949 -1.5707963267949 0 -> xyz=0.048875 -0.0234 0.0094 rpy=1.5708 -1.5708 0
- joint left_knee: axis 0 0 -1 -> 0 0 1; origin xyz=0 -0.162 0 rpy=-3.14159265358979 0 -3.14159265358979 -> xyz=0 -0.137 0 rpy=-3.1416 0 -3.1416
- joint lefthip1motorbody: origin xyz=-0.0234 -0.09425 -0.024125 rpy=0 1.5707963267949 0 -> xyz=-0.0234 -0.08425 -0.024125 rpy=0 1.5708 0
- joint right_ankle: axis 0 0 1 -> 0 0 -1; origin xyz=0 -0.181000000000001 -0.00250000000000579 rpy=0 0 0 -> xyz=0 -0.156 -0.0025 rpy=0 0 0
- joint right_hip1: origin xyz=-0.0234 0.09425 -0.024125 rpy=1.5707963267949 0 1.5707963267949 -> xyz=-0.0234 0.08425 -0.024125 rpy=1.5708 0 1.5708
- joint right_hip2: axis 0 0 1 -> 0 0 -1; origin xyz=0.0233999999999999 -0.048875 0.00940000000000001 rpy=0 1.5707963267949 0 -> xyz=0.0234 -0.048875 0.0094 rpy=0 1.5708 0
- joint right_knee: axis 0 0 1 -> 0 0 -1; origin xyz=0 -0.162000000000005 0 rpy=0 0 0 -> xyz=0 -0.137 0 rpy=0 0 0
